File: 13_TOR_N.kicad_pcb (KiCad board)
At the start: 2 copper layers, 20.3 x 20.3 mm, 15 parts, among them J1 Conn_01x01, J2 Conn_01x01, J3 Conn_01x01, J4 Conn_01x01, J5 Conn_01x01, Q1 FDS8884

Commit message: maj split librairies
Parts:
- H1, H2, H4, H5, H6, H7, H8: footprint Chimere:trou -> Chimere_comps:trou
- J1, J2, J3, J4, J5: footprint Chimere:Castellated_conn -> Chimere_mods:Castellated_conn
