File: 13_TOR_N.sch (KiCad schematic (older format))
At the start: 16 parts, among them J1 Conn_01x01, J2 Conn_01x01, J3 Conn_01x01, J4 Conn_01x01, J5 Conn_01x01, Q1 FDS8884

Commit message: maj split librairies
Parts:
- H1, H2, H3, H4, H5, H6, H7, H8: footprint Chimere:trou -> Chimere_comps:trou
- J1, J2, J3, J4, J5: footprint Chimere:Castellated_conn -> Chimere_mods:Castellated_conn
- Q1: symbol Chimere:FDS6630A -> Chimere_comps:FDS6630A
Changed lines of the file:
@@
 F 0 "J1" H 4380 5117 50  0000 L CNN
 F 1 "Conn_01x01" H 4380 5026 50  0000 L CNN
-F 2 "Chimere:Castellated_conn" H 4300 5075 50  0001 C CNN
+F 2 "Chimere_mods:Castellated_conn" H 4300 5075 50  0001 C CNN
 F 3 "~" H 4300 5075 50  0001 C CNN
 	1    4300 5075
@@
 F 0 "J3" H 4380 5467 50  0000 L CNN
 F 1 "Conn_01x01" H 4380 5376 50  0000 L CNN
-F 2 "Chimere:Castellated_conn" H 4300 5425 50  0001 C CNN
+F 2 "Chimere_mods:Castellated_conn" H 4300 5425 50  0001 C CNN
 F 3 "~" H 4300 5425 50  0001 C CNN
 	1    4300 5425
@@
 F 0 "J2" H 4380 5292 50  0000 L CNN
 F 1 "Conn_01x01" H 4380 5201 50  0000 L CNN
-F 2 "Chimere:Castellated_conn" H 4300 5250 50  0001 C CNN
+F 2 "Chimere_mods:Castellated_conn" H 4300 5250 50  0001 C CNN
 F 3 "~" H 4300 5250 50  0001 C CNN
 	1    4300 5250
@@
 F 0 "J5" H 4380 5667 50  0000 L CNN
 F 1 "Conn_01x01" H 4380 5576 50  0000 L CNN
-F 2 "Chimere:Castellated_conn" H 4300 5625 50  0001 C CNN
+F 2 "Chimere_mods:Castellated_conn" H 4300 5625 50  0001 C CNN
 F 3 "~" H 4300 5625 50  0001 C CNN
 	1    4300 5625
@@
 F 0 "J4" H 4380 4942 50  0000 L CNN
 F 1 "Conn_01x01" H 4380 4851 50  0000 L CNN
-F 2 "Chimere:Castellated_conn" H 4300 4900 50  0001 C CNN
+F 2 "Chimere_mods:Castellated_conn" H 4300 4900 50  0001 C CNN
 F 3 "~" H 4300 4900 50  0001 C CNN
 	1    4300 4900
@@
 F 0 "H1" H 3950 6646 50  0000 L CNN
 F 1 "percage" H 3950 6555 50  0000 L CNN
-F 2 "Chimere:trou" H 3850 6600 50  0001 C CNN
+F 2 "Chimere_comps:trou" H 3850 6600 50  0001 C CNN
 F 3 "~" H 3850 6600 50  0001 C CNN
 	1    3850 6600
@@
 F 0 "H5" H 3950 6921 50  0000 L CNN
 F 1 "percage" H 3950 6830 50  0000 L CNN
-F 2 "Chimere:trou" H 3850 6875 50  0001 C CNN
+F 2 "Chimere_comps:trou" H 3850 6875 50  0001 C CNN
 F 3 "~" H 3850 6875 50  0001 C CNN
 	1    3850 6875
@@
 F 0 "H2" H 4500 6646 50  0000 L CNN
 F 1 "percage" H 4500 6555 50  0000 L CNN
-F 2 "Chimere:trou" H 4400 6600 50  0001 C CNN
+F 2 "Chimere_comps:trou" H 4400 6600 50  0001 C CNN
 F 3 "~" H 4400 6600 50  0001 C CNN
 	1    4400 6600
@@
 F 0 "H6" H 4500 6921 50  0000 L CNN
 F 1 "percage" H 4500 6830 50  0000 L CNN
-F 2 "Chimere:trou" H 4400 6875 50  0001 C CNN
+F 2 "Chimere_comps:trou" H 4400 6875 50  0001 C CNN
 F 3 "~" H 4400 6875 50  0001 C CNN
 	1    4400 6875
@@
 F 0 "H3" H 4975 6646 50  0000 L CNN
 F 1 "percage" H 4975 6555 50  0000 L CNN
-F 2 "Chimere:trou" H 4875 6600 50  0001 C CNN
+F 2 "Chimere_comps:trou" H 4875 6600 50  0001 C CNN
 F 3 "~" H 4875 6600 50  0001 C CNN
 	1    4875 6600
@@
 F 0 "H7" H 4975 6921 50  0000 L CNN
 F 1 "percage" H 4975 6830 50  0000 L CNN
-F 2 "Chimere:trou" H 4875 6875 50  0001 C CNN
+F 2 "Chimere_comps:trou" H 4875 6875 50  0001 C CNN
 F 3 "~" H 4875 6875 50  0001 C CNN
 	1    4875 6875
@@
 F 0 "H4" H 5525 6646 50  0000 L CNN
 F 1 "percage" H 5525 6555 50  0000 L CNN
-F 2 "Chimere:trou" H 5425 6600 50  0001 C CNN
+F 2 "Chimere_comps:trou" H 5425 6600 50  0001 C CNN
 F 3 "~" H 5425 6600 50  0001 C CNN
 	1    5425 6600
@@
 F 0 "H8" H 5525 6921 50  0000 L CNN
 F 1 "percage" H 5525 6830 50  0000 L CNN
-F 2 "Chimere:trou" H 5425 6875 50  0001 C CNN
+F 2 "Chimere_comps:trou" H 5425 6875 50  0001 C CNN
 F 3 "~" H 5425 6875 50  0001 C CNN
 	1    5425 6875
@@
 GND
 $Comp
-L Chimere:FDS6630A Q1
+L Chimere_comps:FDS6630A Q1
 U 1 1 6078CBA9
 P 4550 4075
